File: hardware/schematic/MultiChannel_datalogger.kicad_sch (KiCad schematic)
At the start: 34 parts, among them J1 Conn_01x04_Male, J2 Conn_01x04_Female, J3 Conn_02x08_Top_Bottom, J4 Conn_01x03_Male, J5 Micro_SD_Card, J6 Conn_01x03_Female, Q1 BSS84, Q2 BS170, SW1 RotaryEncoder_Switch, SW2 SW_SPDT_MSM, U1 DS3231MZ, U2 SHT4x, U3 Pico, U4 DS18B20, U5 18650_Boost_TypeC_Module

Commit message: Fix Raspberry Pi Pico footprint library reference
Parts:
- U3: footprint RPi_Pico:RPi_Pico_SMD_TH -> MCU_RaspberryPi_and_Boards:RPi_Pico_SMD_TH
Changed lines of the file:
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@@
 			)
 		)
-		(property "Footprint" "RPi_Pico:RPi_Pico_SMD_TH"
+		(property "Footprint" "MCU_RaspberryPi_and_Boards:RPi_Pico_SMD_TH"
 			(at 121.92 85.09 90)
 			(hide yes)

Commit message: Fix battery voltage measurement circuit
Connections:
- net GND: now reaches BT1.2 (-), Brd1.1 (GND), C2.2, C3.1, C4.2, C5.2, C6.2, C7.1, D1.1 (K), J2.3 (Pin_3), J3.1 (Pin_1), J3.13 (Pin_13), J3.16 (Pin_16), J3.8 (Pin_8), J3.9 (Pin_9), SW1.C, SW1.S2, U1.5 (GND), U3.13 (GND), U3.18 (GND), U3.23 (GND), U3.28 (GND), U3.3 (GND), U3.38 (GND), U3.42 (GND), U3.8 (GND)
- net GND: now also BT2.2 (-), C8.2, J5.6 (VSS), Q2.3 (S), R3.2, R6.2, U5.2 (VIN-), U5.4 (BAT-), U5.6 (OUT-)
Changed lines of the file:
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@@
 	)
 	(junction
+		(at 149.86 133.35)
+		(diameter 0)
+		(color 0 0 0 0)
+	)
+	(junction
 		(at 81.28 157.48)
 		(diameter 0)
@@
 	(wire
 		(pts
-			(xy 185.42 139.7) (xy 185.42 109.22)
-		)
-		(stroke
-			(width 0)
-			(type default)
-		)
-	)
-	(wire
-		(pts
 			(xy 38.1 154.94) (xy 38.1 161.29)
 		)
@@
 	(polyline
 		(pts
-			(xy 267.97 114.3) (xy 182.88 114.3)
+			(xy 267.97 115.57) (xy 182.88 115.57)
 		)
 		(stroke
@@
 	(wire
 		(pts
+			(xy 149.86 139.7) (xy 149.86 133.35)
+		)
+		(stroke
+			(width 0)
+			(type default)
+		)
+	)
+	(wire
+		(pts
 			(xy 25.4 46.99) (xy 30.48 46.99)
 		)
@@
 	(polyline
 		(pts
-			(xy 182.88 54.61) (xy 182.88 114.3)
+			(xy 182.88 54.61) (xy 182.88 115.57)
 		)
 		(stroke
@@
 	(wire
 		(pts
+			(xy 121.92 133.35) (xy 121.92 135.89)
+		)
+		(stroke
+			(width 0)
+			(type default)
+		)
+	)
+	(wire
+		(pts
 			(xy 54.61 116.84) (xy 54.61 99.06)
 		)
@@
 	(polyline
 		(pts
-			(xy 267.97 54.61) (xy 267.97 114.3)
+			(xy 267.97 54.61) (xy 267.97 115.57)
 		)
 		(stroke
@@
 	(wire
 		(pts
+			(xy 185.42 139.7) (xy 149.86 139.7)
+		)
+		(stroke
+			(width 0)
+			(type default)
+		)
+	)
+	(wire
+		(pts
 			(xy 165.1 88.9) (xy 165.1 134.62)
 		)
@@
 	(wire
 		(pts
+			(xy 185.42 111.76) (xy 185.42 109.22)
+		)
+		(stroke
+			(width 0)
+			(type default)
+		)
+	)
+	(wire
+		(pts
 			(xy 210.82 86.36) (xy 210.82 88.9)
 		)
@@
 		(in_pos_files yes)
 		(dnp no)
-		(fields_autoplaced yes)
 		(property "Reference" "J5"
-			(at 236.855 116.9502 0)
+			(at 219.202 119.38 0)
 			(show_name no)
 			(do_not_autoplace no)
@@
 		)
 		(property "Value" "Micro_SD_Card"
-			(at 236.855 119.4871 0)
+			(at 225.298 149.86 0)
 			(show_name no)
 			(do_not_autoplace no)
@@
 	)
 	(symbol
+		(lib_id "power:GND")
+		(at 121.92 135.89 0)
+		(unit 1)
+		(body_style 1)
+		(exclude_from_sim no)
+		(in_bom yes)
+		(on_board yes)
+		(in_pos_files yes)
+		(dnp no)
+		(property "Reference" "#PWR02"
+			(at 121.92 142.24 0)
+			(hide yes)
+			(show_name no)
+			(do_not_autoplace no)
+			(effects
+				(font
+					(size 1.27 1.27)
+				)
+			)
+		)
+		(property "Value" "GND"
+			(at 125.476 138.43 0)
+			(show_name no)
+			(do_not_autoplace no)
+			(effects
+				(font
+					(size 1.27 1.27)
+				)
+			)
+		)
+		(property "Footprint" ""
+			(at 121.92 135.89 0)
+			(hide yes)
+			(show_name no)
+			(do_not_autoplace no)
+			(effects
+				(font
+					(size 1.27 1.27)
+				)
+			)
+		)
+		(property "Datasheet" ""
+			(at 121.92 135.89 0)
+			(hide yes)
+			(show_name no)
+			(do_not_autoplace no)
+			(effects
+				(font
+					(size 1.27 1.27)
+				)
+			)
+		)
+		(property "Description" "Power symbol creates a global label with name \"GND\" , ground"
+			(at 121.92 135.89 0)
+			(hide yes)
+			(show_name no)
+			(do_not_autoplace no)
+			(effects
+				(font
+					(size 1.27 1.27)
+				)
+			)
+		)
+		(pin "1"
+		)
+		(instances
+			(project "MultiChannel_datalogger"
+				(path "/2d805d8a-8bcb-4b88-b4d8-1ed3d5ce3af6"
+					(reference "#PWR02")
+					(unit 1)
+				)
+			)
+		)
+	)
+	(symbol
 		(lib_id "Device:R")
 		(at 210.82 82.55 0)
@@
 		(in_pos_files yes)
 		(dnp no)
-		(fields_autoplaced yes)
 		(property "Reference" "BT2"
 			(at 221.361 92.3818 0)
@@
 		)
 		(property "Value" "3V7 - 18650"
-			(at 221.361 93.6502 0)
+			(at 217.17 111.252 0)
 			(show_name no)
 			(do_not_autoplace no)
@@
 	)
 	(symbol
+		(lib_id "power:GND")
+		(at 185.42 111.76 0)
+		(unit 1)
+		(body_style 1)
+		(exclude_from_sim no)
+		(in_bom yes)
+		(on_board yes)
+		(in_pos_files yes)
+		(dnp no)
+		(property "Reference" "#PWR01"
+			(at 185.42 118.11 0)
+			(hide yes)
+			(show_name no)
+			(do_not_autoplace no)
+			(effects
+				(font
+					(size 1.27 1.27)
+				)
+			)
+		)
+		(property "Value" "GND"
+			(at 188.976 113.538 0)
+			(show_name no)
+			(do_not_autoplace no)
+			(effects
+				(font
+					(size 1.27 1.27)
+				)
+			)
+		)
+		(property "Footprint" ""
+			(at 185.42 111.76 0)
+			(hide yes)
+			(show_name no)
+			(do_not_autoplace no)
+			(effects
+				(font
+					(size 1.27 1.27)
+				)
+			)
+		)
+		(property "Datasheet" ""
+			(at 185.42 111.76 0)
+			(hide yes)
+			(show_name no)
+			(do_not_autoplace no)
+			(effects
+				(font
+					(size 1.27 1.27)
+				)
+			)
+		)
+		(property "Description" "Power symbol creates a global label with name \"GND\" , ground"
+			(at 185.42 111.76 0)
+			(hide yes)
+			(show_name no)
+			(do_not_autoplace no)
+			(effects
+				(font
+					(size 1.27 1.27)
+				)
+			)
+		)
+		(pin "1"
+		)
+		(instances
+			(project "MultiChannel_datalogger"
+				(path "/2d805d8a-8bcb-4b88-b4d8-1ed3d5ce3af6"
+					(reference "#PWR01")
+					(unit 1)
+				)
+			)
+		)
+	)
+	(symbol
 		(lib_id "Device:R")
 		(at 185.42 102.87 0)
@@
 		(dnp no)
 		(property "Reference" "Q2"
-			(at 213.487 95.6853 0)
+			(at 211.582 100.33 0)
 			(show_name no)
 			(do_not_autoplace no)
@@
 		)
 		(property "Value" "BS170"
-			(at 207.01 111.76 0)
+			(at 207.518 111.252 0)
 			(show_name no)
 			(do_not_autoplace no)
